File: hardware/homectrl-rB/ESP-breakout.kicad_sch (KiCad schematic)
At the start: 24 parts, among them J2 USB_C_Female_USB2_Small, SW1 SW_RESET, SW2 SW_BOOT, U1 ESP32-S3-WROOM-1

Commit message: BOM fix
Parts:
- C16, C37: value 10uF -> 10uF
- C35, C36: value 0.1uF -> 0.1uF
- D9: Comments (none) -> Brand: Wurth Elektronik
- U1: Comments (none) -> Confirmed part number is ESP32-S3-WROOM-1-n16R8, different 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
Changed lines of the file:
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@@
 			)
 		)
-		(property "Value" "10uF "
+		(property "Value" "10uF"
 			(at 167.64 59.1819 0)
 			(effects
@@
 			)
 		)
-		(property "Value" "0.1uF "
+		(property "Value" "0.1uF"
 			(at 64.516 123.444 0)
 			(effects
@@
 			)
 		)
-		(property "Value" "0.1uF "
+		(property "Value" "0.1uF"
 			(at 140.97 62.23 0)
 			(effects
@@
 			)
 		)
-		(property "Comments" ""
+		(property "Comments" "Brand: Wurth Elektronik"
 			(at 39.37 95.25 0)
 			(effects
@@
 			)
 		)
-		(property "Comments" ""
+		(property "Comments" "Confirmed part number is ESP32-S3-WROOM-1-n16R8, different from, not WROOM-1-n16R2"
 			(at 148.59 91.44 0)
 			(effects
@@
 			)
 		)
-		(property "Value" "10uF "
+		(property "Value" "10uF"
 			(at 64.262 128.524 0)
 			(effects
