File: hardware/homectrl-rB/actuation-module.kicad_sch (KiCad schematic)
At the start: 26 parts, among them J6 PUMP0-CONN, J7 PUMP1-CONN, J8 STEP-CONN, Q2 AO3400A, Q3 AO3400A, U8 TMC2209

Commit message: dssadasdas
Parts:
- J6, J7: MPN N/A -> S02B-PASK-2; Purchase No -> Yes, Do Not Assemble
- J8: MPN N/A -> S04B-PASK-2; Purchase No -> Yes
- Q2, Q3: Comments Confirmed AO3400A , brand:AOS,package:SOT-23-3L -> Confirmed AO3400A , brand:AOS,package:SOT-23-3L, and brand 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
Changed lines of the file:
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@@
 			)
 		)
-		(property "Comments" "Confirmed AO3400A  , brand:AOS,package:SOT-23-3L"
+		(property "Comments" "Confirmed AO3400A  , brand:AOS,package:SOT-23-3L, and brand AOS"
 			(at 127 64.77 0)
 			(effects
@@
 			)
 		)
-		(property "MPN" "N/A"
+		(property "MPN" "S02B-PASK-2"
 			(at 118.11 27.94 0)
 			(effects
@@
 			)
 		)
-		(property "Purchase" "No"
+		(property "Purchase" "Yes, Do Not Assemble"
 			(at 118.11 27.94 0)
 			(effects
@@
 			)
 		)
-		(property "MPN" "N/A"
+		(property "MPN" "S04B-PASK-2"
 			(at 207.01 27.94 0)
 			(effects
@@
 			)
 		)
-		(property "Purchase" "No"
+		(property "Purchase" "Yes"
 			(at 207.01 27.94 0)
 			(effects
@@
 			)
 		)
-		(property "Comments" "Confirmed AO3400A  , brand:AOS,package:SOT-23-3L"
+		(property "Comments" "Confirmed AO3400A  , brand:AOS,package:SOT-23-3L, and brand AOS"
 			(at 171.45 64.77 0)
 			(effects
@@
 			)
 		)
-		(property "MPN" "N/A"
+		(property "MPN" "S02B-PASK-2"
 			(at 86.36 27.94 0)
 			(effects
@@
 			)
 		)
-		(property "Purchase" "No"
+		(property "Purchase" "Yes, Do Not Assemble"
 			(at 86.36 27.94 0)
 			(effects
