File: hardware/homectrl-rB/sensor-module.kicad_sch (KiCad schematic)
At the start: 27 parts, among them J3 SMS-CONN-0, J4 SMS-CONN-1, J5 ALS_CONN, U5 ADS1115IDGS, U6 SI2301, U7 SI2301, U9 TPD2E001DRLR

Commit message: dssadasdas
Parts:
- J3, J4: MPN N/A -> S03B-PASK-2; Purchase No -> Yes
- J5: MPN N/A -> S04B-PASK-2; Purchase No -> Yes
Changed lines of the file:
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@@
 			)
 		)
-		(property "MPN" "N/A"
+		(property "MPN" "  S03B-PASK-2"
 			(at 55.88 55.88 0)
 			(effects
@@
 			)
 		)
-		(property "Purchase" "No"
+		(property "Purchase" "Yes"
 			(at 55.88 55.88 0)
 			(effects
@@
 			)
 		)
-		(property "MPN" "N/A"
+		(property "MPN" "S04B-PASK-2"
 			(at 114.3 53.34 0)
 			(effects
@@
 			)
 		)
-		(property "Purchase" "No"
+		(property "Purchase" "Yes"
 			(at 114.3 53.34 0)
 			(effects
@@
 			)
 		)
-		(property "MPN" "N/A"
+		(property "MPN" "  S03B-PASK-2"
 			(at 81.28 55.88 0)
 			(effects
@@
 			)
 		)
-		(property "Purchase" "No"
+		(property "Purchase" "Yes"
 			(at 81.28 55.88 0)
 			(effects
