File: hardware/homectrl-rB/power-module.kicad_sch (KiCad schematic)
At the start: 38 parts, among them J1 Barrel_Jack, Q1 DMP6023LE-13, U2 TPS5405DR, U3 ID_LM66100DCKR, U4 ID_LM66100DCKR

Commit message: swap connector in progress
Parts:
- C1: value 100uF 35V -> 100uF
- C10: value 10uF 16V -> 10uF
- C11, C12: value 1uF 12V -> 1uF
- C13: value 0.1uF 25V -> 0.1uF
- C2: value 10uF 25V -> 10uF
- C3: value 47 nF 50V -> 47 nF
- C4: value 3.3nF 16V -> 3.3nF
- C5: value 47nF 25V -> 47nF
- C6: value 47uF 16V -> 47uF
- C7: value 0.47uF 16V -> 0.47uF
- C8: value 22uF 16V -> 22uF
- C9: value 47uF 12V -> 47uF
- D1: value SS14 -> SS24
- D2: Comments (none) -> Littlefuse
- D3: Comments (none) -> diotek
- R3: MPN (none) -> ERJ-2RKF1003X

Commit message: BOM fix
Parts:
- C1: value 100uF -> 100uF
- C10, C2: value 10uF -> 10uF
- C11, C12: value 1uF -> 1uF
- C13: value 0.1uF -> 0.1uF
- C3: value 47 nF -> 47 nF
- C4: value 3.3nF -> 3.3nF
- C5: value 47nF -> 47nF
- C6, C9: value 47uF -> 47uF
- C7: value 0.47uF -> 0.47uF
- C8: value 22uF -> 22uF
Changed lines of the file:
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@@
 			)
 		)
-		(property "Value" "22uF "
+		(property "Value" "22uF"
 			(at 144.526 94.742 0)
 			(effects
@@
 			)
 		)
-		(property "Value" "47uF "
+		(property "Value" "47uF"
 			(at 82.55 140.9699 0)
 			(effects
@@
 			)
 		)
-		(property "Value" "47nF "
+		(property "Value" "47nF"
 			(at 24.638 102.108 0)
 			(effects
@@
 			)
 		)
-		(property "Value" "47uF "
+		(property "Value" "47uF"
 			(at 267.97 64.7699 0)
 			(effects
@@
 			)
 		)
-		(property "Value" "3.3nF "
+		(property "Value" "3.3nF"
 			(at 101.092 101.346 90)
 			(effects
@@
 			)
 		)
-		(property "Value" "10uF "
+		(property "Value" "10uF"
 			(at 116.586 50.8 0)
 			(effects
@@
 			)
 		)
-		(property "Value" "1uF "
+		(property "Value" "1uF"
 			(at 186.182 69.088 0)
 			(effects
@@
 			)
 		)
-		(property "Value" "10uF "
+		(property "Value" "10uF"
 			(at 126.492 94.996 0)
 			(effects
@@
 			)
 		)
-		(property "Value" "0.1uF "
+		(property "Value" "0.1uF"
 			(at 144.272 100.076 0)
 			(effects
@@
 			)
 		)
-		(property "Value" "1uF "
+		(property "Value" "1uF"
 			(at 186.182 50.292 0)
 			(effects
@@
 			)
 		)
-		(property "Value" "100uF "
+		(property "Value" "100uF"
 			(at 90.932 53.34 90)
 			(effects
@@
 			)
 		)
-		(property "Value" "47 nF "
+		(property "Value" "47 nF"
 			(at 35.814 118.364 90)
 			(effects
@@
 			)
 		)
-		(property "Value" "0.47uF "
+		(property "Value" "0.47uF"
 			(at 126.492 99.822 0)
 			(effects
