File: hardware/homectrl-v2/homectrl-v2.kicad_sch (KiCad schematic)
At the start: 57 parts, among them J1 Barrel_Jack, Q1 DMP6023LE-13, Q2 2N7002, U1 TPS5405DR, U2 AMS1117-3.3, U3 DMP4065S-7, U4 ESP32-S3-WROOM-1

Commit message: sch work
Parts:
- added C14, C17: 0.1uF, Capacitor_SMD:C_0402_1005Metric, symbol Device:C
- added C16: 10uF, Capacitor_SMD:C_0603_1608Metric, symbol Device:C
- added C18, C19: C, symbol Device:C
- added D5, D9: D, symbol Device:D
- added J2: PUMP1_CONN, symbol Connector_Generic:Conn_01x02
- added J3: PUMP2_CONN, symbol Connector_Generic:Conn_01x02
- added J4: STEP_CONN, symbol Connector_Generic:Conn_01x04
- added Q3, Q4: PMOS, symbol Simulation_SPICE:PMOS
- added R14, R9: 10k, Resistor_SMD:R_0402_1005Metric, symbol Device:R
- added SW1: S3_RESET_SW, symbol Switch:SW_Push
- added SW2: S3_BOOT_SW, symbol Switch:SW_Push
- added U5: TMC2209, QFN28_5X5_TRI, symbol TMC2209:TMC2209
Connections:
- net +3V3: now also U4.2 (3V3), C14.1, C16.1, R14.2, R9.2
- net GND: now also U4.1 (GND), U4.40 (GND), U4.41 (GND), C14.2, C16.2, C17.2, SW1.2, SW2.2
- net S3_BOOT: now reaches U4.27 (IO0)
- net S3_BOOT: now also R14.1, SW2.1
- net S3_EN: now reaches U4.3 (EN)
- net S3_EN: now also C17.1, R9.1, SW1.1
- new net PUMP1_N: C18.2, D5.2 (A), J2.2 (Pin_2)
- new net PUMP1_P: C18.1, D5.1 (K), J2.1 (Pin_1)
- new net PUMP2_N: C19.2, D9.2 (A), J3.2 (Pin_2)
- new net PUMP2_P: C19.1, D9.1 (K), J3.1 (Pin_1)
- new net STEP_1A: J4.1 (Pin_1)
- new net STEP_1B: J4.2 (Pin_2)
- new net STEP_2A: J4.3 (Pin_3)
- new net STEP_2B: J4.4 (Pin_4)
- no-connect marks 0 -> 2
Other:
- note added: "*place adjacent to S3 PINS 1&2"
- note added: "+"
- note added: "Actuator Inputs"
- note added: "S3 Decoupling"
- note added: "S3 Mode Select"
- moved on the sheet: U4

Commit message: entry circuits
Parts:
- added BZ1: SMT-0540-S-R, SMT-0540-S-R:XDCR_SMT-0540-S-R, symbol SMT-0540-S-R:SMT-0540-S-R
- added C20, C21: 0.1uF, Capacitor_SMD:C_0402_1005Metric, symbol Device:C
- added D11: WIFI_LED, LED_SMD:LED_0603_1608Metric, symbol Device:LED
- added D12: DBG_LED, LED_SMD:LED_0603_1608Metric, symbol Device:LED
- added D13: 1N4148W, Diode_SMD:D_SOD-123, symbol Device:D
- added D14: SYS_LED, LED_SMD:LED_WS2812B-Mini_PLCC4_3.5x3.5mm, symbol LED:WS2812B
- added J5: USB_C_CONN, Connector_USB:USB_C_Receptacle_G-Switch_GT-USB-7010ASV, symbol USB_C:USB_C_Female_USB2_Small
- added J6: SMS1_CONN, symbol Connector_Generic:Conn_01x04
- added J7: SMS2_CONN, symbol Connector_Generic:Conn_01x04
- added J8: FSW1_CONN, symbol Connector_Generic:Conn_01x02
- added J9: FSW2_CONN, symbol Connector_Generic:Conn_01x02
- added Q5: AO3400A, Package_TO_SOT_SMD:SOT-23, symbol Transistor_FET:2N7002
- added R16: 200, Resistor_SMD:R_0402_1005Metric, symbol Device:R
- added R17: 330, Resistor_SMD:R_0402_1005Metric, symbol Device:R
- added R18: 150, Resistor_SMD:R_0402_1005Metric, symbol Device:R
- added R19: 10k, Resistor_SMD:R_0402_1005Metric, symbol Device:R
- added R20, R21: 5.1k, Resistor_SMD:R_0603_1608Metric, symbol Device:R
- added U6: ADS1115IDGS, Package_SO:TSSOP-10_3x3mm_P0.5mm, symbol Analog_ADC:ADS1115IDGS
- added U8, U9: TPD2E001DRLR, TPD2E001DRLR:SOT50P160X60-5N, symbol TPD2E001DRLR:TPD2E001DRLR
Connections:
- net +3V3: now also BZ1.LEAD+, C20.1, C21.1, D13.1 (K), D14.1 (VDD)
- net 5V_USB: now also J5.A4 (VBUS), J5.A9 (VBUS), J5.B4 (VBUS), J5.B9 (VBUS)
- net GND: now also C20.2, C21.2, D11.1 (K), D12.1 (K), D14.3 (VSS), J5.A1 (GND), J5.A12 (GND), J5.B1 (GND), J5.B12 (GND), J5.S1 (SHIELD), Q5.2 (S), R19.1, R20.2, R21.2
- new net: Q5.1 (G), R16.1, R19.2
- new net: BZ1.LEAD-, D13.2 (A), Q5.3 (D)
- new net: J5.B5 (CC2), R21.1
- new net: J5.A5 (CC1), R20.1
- new net: D11.2 (A), R17.2
- new net: D12.2 (A), R18.2
- new net BUZZ_EN: R16.2
- new net DBG_LED: R17.1
- new net RGB_DATA: D14.4 (DIN)
- new net USB_N: J5.A7 (D-), J5.B7 (D-)
- new net USB_P: J5.A6 (D+), J5.B6 (D+)
- new net WIFI_LED: R18.1
- no-connect marks 2 -> 5
Other:
- note added: "Analog Digital Conversion"
- note added: "Buzzer Driver"
- note added: "LED Diagnosis & Indication"
- note added: "Sensor Inputs"
- note added: "Switch Inputs"
- note added: "USB Connector"
- note added: "Vf = 2.1V, R = 68, If = 0.02A * 150 selected for dimness"
- note added: "Vf = 2.8V, R = 100, If = 0.005A * 330 selected for dimness"
- note added: "flyback diode to protect against inductive spikes"
- company: (none) -> Jeevan Sanchez
- title: (none) -> homectrl V2
- moved on the sheet: C18, C19, D5, D9, J2, J3, J4, Q3, Q4, U5

Commit message: peirpheral circuit work
Parts:
- removed Q3, Q4: PMOS, symbol Simulation_SPICE:PMOS
- removed U9: TPD2E001DRLR, TPD2E001DRLR:SOT50P160X60-5N, symbol TPD2E001DRLR:TPD2E001DRLR
- added C22, C23, C24: 0.1uF, Capacitor_SMD:C_0402_1005Metric, symbol Device:C
- added C25: 10uF, Capacitor_SMD:C_0805_2012Metric, symbol Device:C
- added C26, C27, C30, C31: 0.1uF, Capacitor_SMD:C_0402_1005Metric, symbol Device:C_Small
- added C28, C29, C32, C33: 1nF, Capacitor_SMD:C_0402_1005Metric, symbol Device:C_Small
- added Q3, Q4: NMOS, symbol Simulation_SPICE:NMOS
- added R22, R24: 200, Resistor_SMD:R_0402_1005Metric, symbol Device:R
- added R23, R25: 10k, Resistor_SMD:R_0603_1608Metric, symbol Device:R
- added R26: 10k, Resistor_SMD:R_0402_1005Metric, symbol Device:R
- added R27, R28: 330, Resistor_SMD:R_0402_1005Metric, symbol Device:R
- added U7: TPD4E001DRLR, DRL6, symbol TPD4E001DRLR:TPD4E001DRLR
- J7: value SMS2_CONN -> ALS_CONN
- R13: footprint Resistor_SMD:R_0603_1608Metric -> Resistor_SMD:R_0402_1005Metric
Connections:
- net PUMP2_P is gone; now on net PUMP1_P: C19.1, D9.1 (K), J3.1 (Pin_1)
- net VPMP is gone; now on net PUMP1_P: R15.2, U3.3 (D)
- net +3V3: now also J6.2 (Pin_2), J7.2 (Pin_2), J7.3 (Pin_3), J7.4 (Pin_4), U6.10 (SCL), U6.8 (VDD), U6.9 (SDA), U8.1 (VCC), C24.1, C25.2, C26.2, C27.2, C31.2, R26.1, U7.4 (IO3), U7.5 (IO4)
- net GND: now also J6.1 (Pin_1), J7.1 (Pin_1), J8.1 (Pin_1), J9.1 (Pin_1), U8.4 (GND), C22.2, C23.2, C26.1, C27.1, C28.2, C29.2, C31.1, C32.1, C33.1, Q3.3 (S), Q4.3 (S), R23.1, R25.1
- net PUMP1_N: now also Q3.1 (D)
- net PUMP1_P: now also C22.1, C23.1
- net PUMP2_N: now also Q4.1 (D)
- net USB_N: now also U4.4 (IO4)
- net USB_P: now also U4.5 (IO5)
- net at U6.1 (ADDR): now also U6.3 (GND), C24.2, C25.1
- net ADC_ALERT: now reaches U6.2 (ALERT/RDY)
- net ADC_ALERT: now also R26.2
- net SMS1_DATA: now reaches U6.4 (AIN0)
- net SMS1_DATA: now also J6.3 (Pin_3), J6.4 (Pin_4), U6.5 (AIN1), C28.1, C29.1, C30.1, U7.1 (IO1), U7.2 (IO2), U7.3 (GND)
- net at J9.2 (Pin_2): now also R28.1
- net at J8.2 (Pin_2): now also R27.1
- net FSW1_SIG: now reaches U8.3 (IO1)
- net FSW1_SIG: now also C32.2, R27.2
- net FSW2_SIG: now reaches U8.5 (IO2)
- net FSW2_SIG: now also C33.2, R28.2
- new net: C30.2, U7.6 (VCC)
- new net: Q3.2 (G), R22.2, R23.2
- new net: Q4.2 (G), R24.2, R25.2
- new net PUMP1_GATE: R22.1
- new net PUMP2_GATE: R24.1
- no-connect marks 5 -> 7
Other:
- note added: "I2C Pullups"
- moved on the sheet: C18, C19, D5, D9, J2, J3, J4, U5, U6, U8

Commit message: tmc2209 wiring
Parts:
- added C34: 100uF, symbol Device:C_Polarized
- added C35, C36, C37, C39: 0.1uF, Capacitor_SMD:C_0402_1005Metric, symbol Device:C
- added C38: 22nF, Capacitor_SMD:C_0402_1005Metric, symbol Device:C_Small
- added C40: 2.2uF, symbol Device:C
- added R29: 0.11, Resistor_SMD:R_0402_1005Metric, symbol Device:R
- added R30: 0.11, symbol Device:R
- added R31: 1k, Resistor_SMD:R_0402_1005Metric, symbol Device:R
Connections:
- net +3V3: now also U5.15 (VCC_IO), C39.1
- net GND: now also U5.10 (MS2_AD1), U5.13 (CLK), U5.18 (GND), U5.20 (STDBY), U5.3 (GND), U5.9 (MS1_AD0), C39.2, C40.1, R29.2, R30.2
- net STEP_1A: now also U5.24 (OA1)
- net STEP_1B: now also U5.26 (OB1)
- net STEP_2A: now also U5.21 (OA2)
- net STEP_2B: now also U5.1 (OB2)
- net STEP_DIAG: now reaches U5.11 (DIAG)
- net S3_TXD: now reaches U5.14 (PDN_UART)
- net S3_TXD: now also R31.1
- net MTR_STEP: now reaches U5.16 (STEP)
- net MTR_DIR: now reaches U5.19 (DIR)
- net STEP_ENN: now reaches U5.2 (ENN)
- net at U5.22 (VS): now also U5.28 (VS), C34.1, C35.2, C36.2, C37.1
- net at U5.23 (BRA): now also R30.1
- net at U5.27 (BRB): now also R29.1
- net at U5.29 (GND): now also C34.2, C35.1, C36.1
- net at U5.4 (CPO): now also C38.2
- net at U5.5 (CPI): now also C38.1
- net at U5.6 (VCP): now also C37.2
- net at U5.8 (5VOUT): now also C40.2
- new net S3_RXD: R31.2
- no-connect marks 7 -> 10

Commit message: power calculations
Parts:
- removed Q1: DMP6023LE-13, Package_TO_SOT_SMD:SOT-223, symbol Transistor_FET:FQP27P06
- removed Q3, Q4: NMOS, symbol Simulation_SPICE:NMOS
- removed U2: AMS1117-3.3, Package_TO_SOT_SMD:SOT-223-3_TabPin2, symbol Regulator_Linear:AMS1117
- added C41, C43: 0.1uF, Capacitor_SMD:C_0402_1005Metric, symbol Device:C
- added C42: 22uF, Capacitor_SMD:C_0805_2012Metric, symbol Device:C
- added C44: 22uF, Capacitor_SMD:C_1206_3216Metric, symbol Device:C
- added Q4, Q6: DMN3032LE-13, SOT230P700X180-4N, symbol DMN3032LE-13:DMN3032LE-13
- added R32, R33: 10k, Resistor_SMD:R_0402_1005Metric, symbol Device:R
- added R34, R35: 4.7k, Resistor_SMD:R_0402_1005Metric, symbol Device:R
- added U2: MCP1826S, Package_TO_SOT_SMD:SOT-223-3_TabPin2, symbol Regulator_Linear:MCP1826S
- added U9: SI2347DS-T1-GE3, SOT_7DS-T1-GE3_VIS, symbol Si2347DS:SI2347DS-T1-GE3
- C10, C12, C15, C7, C9: footprint Capacitor_SMD:C_0603_1608Metric -> Capacitor_SMD:C_0402_1005Metric
- C11: footprint Capacitor_SMD:C_0805_2012Metric -> Capacitor_SMD:C_1206_3216Metric
- C16: footprint Capacitor_SMD:C_0603_1608Metric -> Capacitor_SMD:C_0805_2012Metric
- C18, C19: value C -> 0.1uF; footprint (none) -> Capacitor_SMD:C_0402_1005Metric
- C3: value ~ -> 10uF; footprint (none) -> Capacitor_SMD:C_0805_2012Metric; LCSC C15850 -> (none)
- C32, C33: value 1nF -> 0.1uF
- C34: footprint (none) -> EEH_ZK1V101XP:CAP_EEHZK1V101XP
- C4: value ~ -> 10nF; footprint (none) -> Capacitor_SMD:C_0402_1005Metric; LCSC C15195 -> (none)
- C40: footprint (none) -> Capacitor_SMD:C_0402_1005Metric
- C5: value ~ -> 0.1uF; footprint (none) -> Capacitor_SMD:C_0402_1005Metric; LCSC C14663 -> (none)
- C6: value ~ -> 22uF; footprint (none) -> Capacitor_SMD:C_0805_2012Metric
- C8: value ~ -> 3.3nF
- D1: value ~ -> SMBJ14A; footprint Diode_SMD:D_SMA -> Diode_SMD:D_SMB
- D2: footprint LED_SMD:LED_0603_1608Metric -> LED_SMD:LED_0805_2012Metric; LCSC (none) -> C2297; MPN 150060GS75000 -> (none); Purchase Yes -> (none)
- D3: value D_Zener -> MMSZ5243BT1G
- D4: value ~ -> SS34; footprint (none) -> Diode_SMD:D_SMB
- D5, D9: value D -> SS14; footprint (none) -> Diode_SMD:D_SMA
- F1: value Polyfuse -> 3A 24V PTC; footprint (none) -> Fuse:Fuse_1812_4532Metric
- FB1: footprint (none) -> Resistor_SMD:R_1206_3216Metric
- J1: footprint (none) -> Connector_BarrelJack:BarrelJack_Horizontal
- J2, J3, J8, J9: footprint (none) -> S02B_PASK_2:CONN2_S02B-PASK-2_JST
- J4, J6, J7: footprint (none) -> S04B_PASK_2:CONN4_S04B-PASK_JST
- L1: value ~ -> 10uH; footprint (none) -> ETQ_P3M100HFN:IND_ETQP3M100HFN
- R1: value ~ -> 4.7k; footprint (none) -> Resistor_SMD:R_0402_1005Metric; LCSC (none) -> C22765
- R10, R11, R20, R21, R23, R25, R5, R6, R7, R8: footprint Resistor_SMD:R_0603_1608Metric -> Resistor_SMD:R_0402_1005Metric
- R12, R15: value 4.7k -> 1k; footprint Resistor_SMD:R_0603_1608Metric -> Resistor_SMD:R_0402_1005Metric
- R2: value ~ -> 100k; footprint Resistor_SMD:R_0402_1005Metric -> Resistor_SMD:R_0805_2012Metric
- R3: value ~ -> 50k; footprint (none) -> Resistor_SMD:R_0402_1005Metric; LCSC C25803 -> (none)
- R30: footprint (none) -> Resistor_SMD:R_0402_1005Metric
- R4: value ~ -> 10k; footprint (none) -> Resistor_SMD:R_0402_1005Metric
- SW1, SW2: footprint (none) -> TACT_TS1185:SW_5-B-B-B-A_XKB
- U7: footprint DRL6 -> TPD2E001DRLR:SOT50P160X60-5N
Connections:
- net +3V3: now also R32.1, R33.1, R34.1, R35.1, U2.3 (VO); no longer J7.3 (Pin_3), J7.4 (Pin_4), U6.10 (SCL), U6.9 (SDA), U7.4 (IO3), U7.5 (IO4)
- net 5V_MUX: now also C44.1, U2.1 (VI)
- net 5V_PLUG: now also C42.1, C43.1
- net FSW1_SIG: now also R33.2
- net FSW2_SIG: now also R32.2
- net GND: now also C30.2, C34.2, C35.1, C36.1, C4.1, R3.2, U5.29 (GND), U7.3 (GND), C42.2, C43.2, C44.2, Q4.3 (S), Q6.3 (S), U2.2 (GND); no longer C22.2, C23.2
- net PUMP1_N: now also C22.2, Q4.2 (D_1), Q4.4 (D_2)
- net PUMP2_N: now also C23.2, Q6.2 (D_1), Q6.4 (D_2)
- net SMS1_DATA: no longer C29.1, C30.1, J6.4 (Pin_4), U6.5 (AIN1), U7.2 (IO2), U7.3 (GND)
- net VPLUG: now also C41.1
- net at U7.6 (VCC): now also C30.1; no longer C30.2
- net at D1.1 (A1), F1.2, R1.2: now also U9.3
- net at C1.2, C2.1, D3.2 (A)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: now also C41.2, U9.1
- net at R22.2, R23.2: now also Q4.1 (G)
- net at R24.2, R25.2: now also Q6.1 (G)
- net at C1.1, D3.1 (K), FB1.1: now also U9.2
- new net I2C_CLK: J7.4 (Pin_4), R35.2, U6.10 (SCL), U7.5 (IO4)
- new net I2C_DTA: J7.3 (Pin_3), R34.2, U6.9 (SDA), U7.4 (IO3)
- new net SMS2_DATA: C29.1, J6.4 (Pin_4), U6.5 (AIN1), U7.2 (IO2)
Other:
- note added: "** For NEMA 17 Phase Resistance = 2 ohm 1 A RMS set via TMC2209 Efficiency = 85% Istep = Pstep / VPLUG Pstep = (2 x (1 A)^2 * 2 ohm) / 0.85 = 4.7 W Istep = 4.7W / 12V = 0.4 A"
- note added: "1.25 x Net Current Greater than 12V"
- note added: "Actuator Calculations"
- note added: "Buck Converter Calculations"
- note added: "FB diode specs: PIV > 24V If > 0.3 A"
- note added: "Fuse Rating"
- note added: "I = 3 A"
- note added: "I > 2.5 A"
- note added: "MOSFET specs for Pump Drivers"
- note added: "Manually set ROSC; by default, fsw = 120 kHz With 200k resistor, fsw ≈ 525 kHz (Inverse) Css (nF) = (tss (ms) * Iss (uA) / Vref (V) Iss = 2uA, Vref = 0.8V from datasheet Target start time of 5ms Css = 5 * 2.5 = 12.5 nf ≈ 10 nF (std value) Schottky Catch Diode Must be > Vin; V > 13V, Handle 2A output current Inductor L = ((Vout)*(Vin - Vout)) / ((Vin)(fsw)(ΔIl) - Target ΔIl = 0.6A L = ((5V)*(12-5)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"
- note added: "Net Current = Ipmp + Istep + Iperiph = 0.6A + 0.4A + 1 A = 2 A"
- note added: "SI2347DS chosen for RPP - Vds > (2x13V) ≈ 30V - Id > Inet ≈ 5A - P = I^2 * R = (3)^2 * (0.042) = 0.378 W (heat)"
- note added: "TVS diode standoff @ 14V, breakdown @ 15.6V, clamps @ 23.2V"
- note added: "VPLUG Buck Conversion"
- note added: "Vds > VPMP. More headroom the better; aiming for 30+ V. (VPMP = 12V) Id > 0.3A (I of pump) 1A - 5A Rds < 0.5 ohm To minimize heat dissipation; P (Heat) = I^2 x Rds"
- note added: "Zener Diode rated for 13V, clamps gate voltage at 13V in case of spike"
- note added: "π-Filter Ferrite Bead Isat = 1.5 * Inet Isat = 1.5 * 2 A ≈ 3 A Low heat dissipation. DCR < 50mohm Isat = P = I^2 * DCR = (5A)^2 * (0.01) = 0.25 W (heat)"
- moved on the sheet: BZ1, C1, C10, C11, C12, C13, C15, C18, C19, C2, C20, C21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

Commit message: power layout
Parts:
- added C45: 100uF, EEH_ZK1V101XP:CAP_EEHZK1V101XP, symbol Device:C_Polarized
- C1: footprint EEE_FK1V101P:CAP_EEEFK1V101P -> EEH_ZK1V101XP:CAP_EEHZK1V101XP
- C11: footprint Capacitor_SMD:C_1206_3216Metric -> Capacitor_SMD:C_0402_1005Metric
- C13, C44: footprint Capacitor_SMD:C_1206_3216Metric -> Capacitor_SMD:C_0805_2012Metric
- D1: value SMBJ14A -> SMAJ14A; footprint Diode_SMD:D_SMB -> Diode_SMD:D_SMA
- D2: footprint LED_SMD:LED_0805_2012Metric -> Diode_SMD:D_0603_1608Metric
- D4: footprint Diode_SMD:D_SMB -> Nexperia_CFP3_SOD-123W
- L1: footprint ETQ_P3M100HFN:IND_ETQP3M100HFN -> L_Changjiang_FNR6045S
- U4: footprint RF_Module:ESP32-S3-WROOM-1 -> ESP32-S3-WROOM-1-N16R2:XCVR_ESP32-S3-WROOM-1-N16R2
Connections:
- net 5V_BATT is gone; now on net 5V_PLUG: C7.2, UE1.1 (VIN)
- net GND: now also C1.2, C2.1, C41.2, D3.2 (A), R2.1, U9.1
- net VPLUG: now also C34.1, C35.2, C36.2, C37.1, U5.22 (VS), U5.28 (VS)
- net at F1.1, J1.1: now also R1.2
- net at D1.1 (A1), F1.2, U9.3: no longer R1.2
Other:
- moved on the sheet: D1, D2, F1, R1

Commit message: fet fix
Parts:
- removed C22, C23: 0.1uF, Capacitor_SMD:C_0402_1005Metric, symbol Device:C
Connections:
- net PUMP1_P renamed VPMP

Commit message: experimenting w connectors
Parts:
- removed C45: 100uF, EEH_ZK1V101XP:CAP_EEHZK1V101XP, symbol Device:C_Polarized
- C16, C25: footprint Capacitor_SMD:C_0805_2012Metric -> Capacitor_SMD:C_0402_1005Metric
- J2, J3, J8, J9: footprint S02B_PASK_2:CONN2_S02B-PASK-2_JST -> JST_XH_B2B-XH-A_1x02_P2.50mm_Vertical
- J4, J6, J7: footprint S04B_PASK_2:CONN4_S04B-PASK_JST -> JST_XH_B4B-XH-A_1x04_P2.50mm_Vertical
- U7: footprint TPD2E001DRLR:SOT50P160X60-5N -> Package_TO_SOT_SMD:Texas_R-PDSO-N6_DRL-6
Connections:
- net +3V3: now also C30.1, U7.6 (VCC)
- net GND: now also C24.2, C25.1, U6.1 (ADDR), U6.3 (GND)
- net I2C_CLK: now also U7.4 (IO3); no longer U7.5 (IO4)
- net I2C_DTA: now also U7.5 (IO4); no longer U7.4 (IO3)
- net SMS1_DATA: now also U7.2 (IO2); no longer U7.1 (IO1)
- net SMS2_DATA: now also U7.1 (IO1); no longer U7.2 (IO2)
- net USB_N: now also U4.6 (IO6); no longer U4.4 (IO4)
- net USB_P: now also U4.7 (IO7); no longer U4.5 (IO5)
