File: hardware/homectrl-v2/homectrl-v2.kicad_sch (KiCad schematic)
At the start: 133 parts, among them J1 Barrel_Jack, J2 PUMP1_CONN, J3 PUMP2_CONN, J4 STEP_CONN, J5 USB_C_CONN, J6 SMS1_CONN, J7 ALS_CONN, J8 FSW1_CONN, Q1 AO3407A, Q2 2N7002, Q3 AO3400A, Q4 AO3400A, Q5 AO3400A, SW1 S3_RESET_SW, SW2 S3_BOOT_SW, U1 TPS5405DR, U2 MCP1826S, U3 DMP4065S-7, U4 ESP32-S3-WROOM-1, U5 TMC2209, U7 TPD4E001DRLR, U8 TPD2E001DRLR, U9 SI2347DS-T1-GE3

Commit message: silkscreen
Parts:
- added H1, H2: MountingHole, MountingHole:MountingHole_2.2mm_M2, symbol Mechanical:MountingHole
- C11, C16: footprint Capacitor_SMD:C_0402_1005Metric -> Capacitor_SMD:C_0603_1608Metric; LCSC (none) -> C96446
- C22, C23: LCSC C913517 -> C96446
- C25: value 10uF -> 0.1uF
- C42, C6: LCSC (none) -> C45783
- L1: LCSC (none) -> C360734
- TP5: footprint TestPoint_Pad_D1.0mm -> TestPoint_Pad_D1.0mm
Other:
- note added: "ESP32-S3"
- note added: "Mounting Holes"
- moved on the sheet: C14, C16, C17, R14, R34, R35, R9, SW1, SW2

Commit message: prod
Parts:
- added TP7: VPLUG_TP_PAD, TestPoint:TestPoint_Pad_1.0x1.0mm, symbol Connector:TestPoint
- added TP9: GND_B_PAD, TestPoint:TestPoint_Pad_1.0x1.0mm, symbol Connector:TestPoint
- C25: LCSC (none) -> C77020
- D14: now fitted
- TP5: value VPLUG_TP_PAD -> VPLUG_TP_DRILL; footprint TestPoint_Pad_D1.0mm -> TestPoint:TestPoint_THTPad_D1.0mm_Drill0.5mm
Connections:
- net GND: now also D1.2 (A2), J1.2, TP9.1; no longer D3.2 (A), U9.1
- net at C1.1, D3.1 (K), FB1.1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: now also TP7.1
- new net: D3.2 (A), R2.2, U9.1

Commit message: cleanup
Other:
- note removed: "Actuator Calculations"
- moved on the sheet: BZ1, C1, C10, C11, C12, C13, C14, C15, C16, C17, C18, C19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

Commit message: add imgs
Parts:
- BZ1, C1, C34, D1, D5, D9, F1, FB1, J1, J2, J3, J4, J6, J7, J8: now fitted
Changed lines of the file:
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@@
 		(in_bom yes)
 		(on_board yes)
-		(dnp yes)
+		(dnp no)
 		(property "Reference" "J1"
 			(at 49.784 59.69 0)
@@
 		(in_bom yes)
 		(on_board yes)
-		(dnp yes)
+		(dnp no)
 		(property "Reference" "J7"
 			(at 342.392 271.018 90)
@@
 		(in_bom yes)
 		(on_board yes)
-		(dnp yes)
+		(dnp no)
 		(fields_autoplaced yes)
 		(property "Reference" "J2"
@@
 		(in_bom yes)
 		(on_board yes)
-		(dnp yes)
+		(dnp no)
 		(property "Reference" "J4"
 			(at 449.072 48.768 90)
@@
 		(in_bom yes)
 		(on_board yes)
-		(dnp yes)
+		(dnp no)
 		(fields_autoplaced yes)
 		(property "Reference" "BZ1"
@@
 		(in_bom yes)
 		(on_board yes)
-		(dnp yes)
+		(dnp no)
 		(fields_autoplaced yes)
 		(property "Reference" "J3"
@@
 		(in_bom yes)
 		(on_board yes)
-		(dnp yes)
+		(dnp no)
 		(property "Reference" "D1"
 			(at 93.472 66.294 90)
@@
 		(in_bom yes)
 		(on_board yes)
-		(dnp yes)
+		(dnp no)
 		(property "Reference" "J6"
 			(at 309.372 271.018 90)
@@
 		(in_bom yes)
 		(on_board yes)
-		(dnp yes)
+		(dnp no)
 		(fields_autoplaced yes)
 		(property "Reference" "D5"
@@
 		(in_bom yes)
 		(on_board yes)
-		(dnp yes)
+		(dnp no)
 		(fields_autoplaced yes)
 		(property "Reference" "J8"
@@
 		(in_bom yes)
 		(on_board yes)
-		(dnp yes)
+		(dnp no)
 		(property "Reference" "FB1"
 			(at 165.608 46.99 90)
@@
 		(in_bom yes)
 		(on_board yes)
-		(dnp yes)
+		(dnp no)
 		(property "Reference" "C1"
 			(at 158.75 50.038 0)
@@
 		(in_bom yes)
 		(on_board yes)
-		(dnp yes)
+		(dnp no)
 		(fields_autoplaced yes)
 		(property "Reference" "D9"
@@
 		(in_bom yes)
 		(on_board yes)
-		(dnp yes)
+		(dnp no)
 		(property "Reference" "C34"
 			(at 530.606 113.284 0)
@@
 		(in_bom yes)
 		(on_board yes)
-		(dnp yes)
+		(dnp no)
 		(property "Reference" "F1"
 			(at 82.55 53.34 90)
