File: hardware/homectrl-v2/homectrl-v2.kicad_pcb (KiCad board)
At the start: 2 copper layers, 134 parts, among them J1 Barrel_Jack, J2 PUMP1_CONN, J3 PUMP2_CONN, J4 STEP_CONN, J5 USB_C_CONN, J6 SMS1_CONN, J7 ALS_CONN, J8 FSW1_CONN, J9 FSW2_CONN, Q1 Si2347DS, Q2 2N7002, Q4 DMN3032LE-13, Q5 AO3400A, Q6 DMN3032LE-13, SW1 S3_RESET_SW, SW2 S3_BOOT_SW, U1 TPS5405DR, U2 MCP1826S, U3 DMP4065S-7, U4 ESP32-S3-WROOM-1, U5 TMC2209, U6 ADS1115IDGS, U7 TPD4E001DRLR, U8 TPD2E001DRLR, U9 SI2347DS-T1-GE3

Commit message: power layout
Parts:
- removed Q1: Si2347DS, Package_TO_SOT_SMD:SOT-223
- added C45: 100uF, EEH_ZK1V101XP:CAP_EEHZK1V101XP, F.Cu at (4.38, 3.58)
- C1: footprint EEE_FK1V101P:CAP_EEEFK1V101P -> EEH_ZK1V101XP:CAP_EEHZK1V101XP
- C11: footprint Capacitor_SMD:C_1206_3216Metric -> Capacitor_SMD:C_0402_1005Metric
- C13, C44: footprint Capacitor_SMD:C_1206_3216Metric -> Capacitor_SMD:C_0805_2012Metric
- D1: value SMBJ14A -> SMAJ14A; footprint Diode_SMD:D_SMB -> Diode_SMD:D_SMA
- D2: footprint LED_SMD:LED_0805_2012Metric -> Diode_SMD:D_0603_1608Metric
- D4: footprint Diode_SMD:D_SMB -> Diode_SMD:Nexperia_CFP3_SOD-123W
- J8, J9: moved to B.Cu
- L1: footprint ETQ_P3M100HFN:IND_ETQP3M100HFN -> Inductor_SMD:L_Changjiang_FNR6045S
- U4: footprint RF_Module:ESP32-S3-WROOM-1 -> ESP32-S3-WROOM-1-N16R2:XCVR_ESP32-S3-WROOM-1-N16R2
- moved J5 198.8 mm to (229.4, 97.1)
- moved U4 181.7 mm to (213.5, 94.5), turned to 180 degrees
- moved C39 119.8 mm to (144.9, 63.1)
- moved C36 118.2 mm to (143.3, 57.3), turned to -90 degrees
- moved C35 116.7 mm to (138.1, 57.4), turned to -90 degrees
- moved D9 116.2 mm to (151.9, 108.3), turned to -90 degrees
- moved D5 115.0 mm to (151.9, 100.3), turned to -90 degrees
- moved C40 112.7 mm to (137.7, 64.7)
- moved C37 111.5 mm to (136.5, 63.1)
- moved C38 111.2 mm to (136.2, 61.5)
- moved Q4 109.4 mm to (173.7, 57.1)
- moved Q6 109.4 mm to (173.7, 65.2)
- moved U3 106.3 mm to (158.7, 40.9)
- moved J6 106.3 mm to (200.4, 73.9), turned to 90 degrees
- moved C1 105.1 mm to (136.3, 42.7), turned to 90 degrees
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Connections:
- C1 pad 2: Net-(D3-A) -> GND
- C2 pad 1: Net-(D3-A) -> GND
- C34 pad 1: Net-(C34-Pad1) -> VPLUG
- C35 pad 2: Net-(C34-Pad1) -> VPLUG
- C36 pad 2: Net-(C34-Pad1) -> VPLUG
- C37 pad 1: Net-(C34-Pad1) -> VPLUG
- C41 pad 2: Net-(D3-A) -> GND
- C7 pad 2: 5V_BATT -> 5V_PLUG
- D3 pad 2: Net-(D3-A) -> GND
- R1 pad 2: Net-(D1-A1) -> Net-(F1-Pad1)
- R2 pad 1: Net-(D3-A) -> GND
- U5 pad 22: Net-(C34-Pad1) -> VPLUG
- U5 pad 28: Net-(C34-Pad1) -> VPLUG
- U9 pad 1: Net-(D3-A) -> GND
- UE1 pad 1: 5V_BATT -> 5V_PLUG

Commit message: experimenting w connectors
Parts:
- removed C45: 100uF, EEH_ZK1V101XP:CAP_EEHZK1V101XP
- removed J9: FSW2_CONN, S02B_PASK_2:CONN2_S02B-PASK-2_JST
- added REF**: JST_XH_S2B-XH-A-1_1x02_P2.50mm_Horizontal, Connector_JST:JST_XH_S2B-XH-A-1_1x02_P2.50mm_Horizontal, F.Cu at (150.4, 72.5)
- added REF**: JST_XH_S4B-XH-A-1_1x04_P2.50mm_Horizontal, Connector_JST:JST_XH_S4B-XH-A-1_1x04_P2.50mm_Horizontal, F.Cu at (150.5, 63.0)
- added REF**: JST_XH_S2B-XH-A-1_1x02_P2.50mm_Horizontal, Connector_JST:JST_XH_S2B-XH-A-1_1x02_P2.50mm_Horizontal, F.Cu at (150.3, 81.7)
- C16, C25: footprint Capacitor_SMD:C_0805_2012Metric -> Capacitor_SMD:C_0402_1005Metric
- C34: moved to B.Cu
- J2, J3: footprint S02B_PASK_2:CONN2_S02B-PASK-2_JST -> Connector_JST:JST_XH_B2B-XH-A_1x02_P2.50mm_Vertical
- J4, J6, J7: footprint S04B_PASK_2:CONN4_S04B-PASK_JST -> Connector_JST:JST_XH_B4B-XH-A_1x04_P2.50mm_Vertical
- J8: footprint S02B_PASK_2:CONN2_S02B-PASK-2_JST -> Connector_JST:JST_XH_B2B-XH-A_1x02_P2.50mm_Vertical; moved to F.Cu
- U7: footprint TPD2E001DRLR:SOT50P160X60-5N -> Package_TO_SOT_SMD:Texas_R-PDSO-N6_DRL-6
- moved C20 218.3 mm to (193.0, 88.4)
- moved C19 170.7 mm to (140.2, 79.9), turned to -90 degrees
- moved C18 166.4 mm to (140.2, 70.5), turned to -90 degrees
- moved R21 153.2 mm to (135.9, 90.0)
- moved R20 152.8 mm to (131.8, 90.0), turned to 180 degrees
- moved C14 147.7 mm to (126.5, 91.2), turned to -90 degrees
- moved R9 144.4 mm to (127.0, 89.5)
- moved C17 143.5 mm to (127.0, 88.5)
- moved C24 139.2 mm to (115.4, 70.2), turned to 180 degrees
- moved C28 135.4 mm to (103.3, 71.8)
- moved C16 135.2 mm to (127.6, 91.2), turned to -90 degrees
- moved R24 134.9 mm to (130.1, 78.0)
- moved R25 134.9 mm to (130.6, 79.7), turned to 90 degrees
- moved C27 134.8 mm to (106.9, 65.2), turned to 90 degrees
- moved C29 133.1 mm to (103.3, 70.5)
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Connections:
- C18 pad 1: PUMP1_P -> VPMP
- C19 pad 1: PUMP1_P -> VPMP
- C24 pad 2: Net-(U6-ADDR) -> GND
- C25 pad 1: Net-(U6-ADDR) -> GND
- C30 pad 1: Net-(U7-VCC) -> +3V3
- D5 pad 1: PUMP1_P -> VPMP
- D9 pad 1: PUMP1_P -> VPMP
- J2 pad 1: PUMP1_P -> VPMP
- J3 pad 1: PUMP1_P -> VPMP
- R15 pad 2: PUMP1_P -> VPMP
- U3 pad 3: PUMP1_P -> VPMP
- U4 pad 4: USB_N -> unconnected-(U4-IO4-Pad4)
- U4 pad 5: USB_P -> unconnected-(U4-IO5-Pad5)
- U4 pad 6: unconnected-(U4-IO6-Pad6) -> USB_N
- U4 pad 7: unconnected-(U4-IO7-Pad7) -> USB_P
- U6 pad 1: Net-(U6-ADDR) -> GND
- U6 pad 3: Net-(U6-ADDR) -> GND
- U7 pad 1: SMS1_DATA -> SMS2_DATA
- U7 pad 2: SMS2_DATA -> SMS1_DATA
- U7 pad 4: I2C_DTA -> I2C_CLK
- U7 pad 5: I2C_CLK -> I2C_DTA
Routing:
- net S3_EN: track 0.00 -> 21.3 mm, vias 0 -> 2
- net USB_P: track 0.00 -> 18.7 mm
- net USB_N: track 0.00 -> 17.9 mm
- net PUMP1_GATE: track 0.00 -> 16.0 mm
- net VPMP_EN: track 0.00 -> 9.53 mm
- net PUMP2_GATE: track 0.00 -> 8.15 mm
- net VPMP: track 0.00 -> 6.71 mm
- net VPLUG: track 0.00 -> 6.19 mm
- net +3V3: track 0.00 -> 5.91 mm
- net Net-(Q2-D): track 0.00 -> 4.08 mm
- net GND: track 0.00 -> 3.73 mm, vias 0 -> 1
- net Net-(Q4-G): track 0.00 -> 2.89 mm
- net Net-(Q6-G): track 0.00 -> 2.86 mm
- net Net-(U5-VCP): track 0.00 -> 2.14 mm
- net Net-(U5-5VOUT): track 0.00 -> 1.85 mm
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Other:
- board outline added: 64 x 64 mm
- board text added: "homectrl"

Commit message: connectot placement
Parts:
- removed REF** (x2): JST_XH_S2B-XH-A-1_1x02_P2.50mm_Horizontal, Connector_JST:JST_XH_S2B-XH-A-1_1x02_P2.50mm_Horizontal
- removed REF**: JST_XH_S4B-XH-A-1_1x04_P2.50mm_Horizontal, Connector_JST:JST_XH_S4B-XH-A-1_1x04_P2.50mm_Horizontal
- C34: moved to F.Cu
- moved J6 79.2 mm to (99.2, 72.0), turned to -70 degrees
- moved J7 78.6 mm to (100.0, 57.1), turned to -100 degrees
- moved J8 68.3 mm to (149.8, 54.4), turned to 120 degrees
- moved J3 54.3 mm to (142.3, 87.4), turned to 45 degrees
- moved J2 49.2 mm to (148.7, 79.7), turned to 60 degrees
- moved J4 46.1 mm to (151.7, 69.5)
- moved C19 44.3 mm to (183.1, 69.1)
- moved D5 44.3 mm to (185.6, 60.2)
- moved D9 44.3 mm to (185.5, 69.5)
- moved Q4 44.3 mm to (178.3, 60.2)
- moved Q6 44.3 mm to (178.2, 69.5)
- moved R22 44.3 mm to (173.1, 57.9)
- moved R23 44.3 mm to (173.6, 59.5)
- moved R24 44.3 mm to (173.0, 67.2)
- moved R25 44.3 mm to (173.5, 68.9)
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Routing:
- net PUMP2_GATE: track 8.15 -> 0.00 mm
- net PUMP1_GATE: track 16.0 -> 12.0 mm
- net VPMP: track 6.71 -> 4.49 mm
- net Net-(Q4-G): track 2.89 -> 1.17 mm
- net VPMP_EN: track 9.53 -> 8.36 mm
Other:
- board text removed: "homectrl"

Commit message: layout work
Parts:
- removed C25: 10uF, Capacitor_SMD:C_0402_1005Metric
- removed C28, C29: 1nF, Capacitor_SMD:C_0402_1005Metric
- removed U6: ADS1115IDGS, Package_SO:TSSOP-10_3x3mm_P0.5mm
- C18, C19: footprint Capacitor_SMD:C_0402_1005Metric -> Capacitor_SMD:C_0603_1608Metric
- C22, C23: value 0.1uF -> 10uF; footprint Capacitor_SMD:C_0402_1005Metric -> Capacitor_SMD:C_0603_1608Metric
- J8: footprint Connector_JST:JST_XH_B2B-XH-A_1x02_P2.50mm_Vertical -> Connector_JST:JST_XH_B3B-XH-AM_1x03_P2.50mm_Vertical
- R27: value 330 -> 1k
- R28: value 330 -> 10k
- R32: value 10k -> 1k
- moved C20 143.0 mm to (53.3, 57.9)
- moved C22 123.9 mm to (142.6, 73.9), turned to 60 degrees
- moved C23 121.3 mm to (139.1, 79.1), turned to 45 degrees
- moved C31 118.1 mm to (142.4, 55.3), turned to 180 degrees
- moved U8 118.0 mm to (144.8, 55.2)
- moved C24 50.5 mm to (65.3, 76.5), turned to 0 degrees
- moved R22 48.1 mm to (128.1, 74.7), turned to 90 degrees
- moved R24 47.8 mm to (127.9, 82.8), turned to 90 degrees
- moved R23 47.4 mm to (128.1, 72.7)
- moved Q4 47.4 mm to (132.8, 73.3)
- moved D9 47.1 mm to (140.6, 83.5), turned to 45 degrees
- moved R25 47.0 mm to (127.9, 80.5), turned to -90 degrees
- moved Q6 46.8 mm to (132.8, 80.7)
- moved C19 44.4 mm to (140.2, 80.2), turned to 45 degrees
- moved D5 42.9 mm to (145.9, 76.4), turned to 60 degrees
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Connections:
- C22 pad 1: PUMP1_P -> VPMP
- C23 pad 1: PUMP1_P -> VPMP
- C24 pad 1: +3V3 -> Net-(C24-Pad1)
- C24 pad 2: GND -> FSW2_SIG
- C32 pad 1: GND -> Net-(C32-Pad1)
- J8 pad 1: GND -> Net-(J8-Pin_1)
- R26 pad 2: ADC_ALERT -> Net-(J8-Pin_1)
- R27 pad 1: Net-(J8-Pin_2) -> Net-(C32-Pad1)
- R27 pad 2: FSW1_SIG -> Net-(J8-Pin_1)
- R28 pad 1: Net-(J9-Pin_2) -> +3V3
- R28 pad 2: FSW2_SIG -> Net-(J8-Pin_2)
- R32 pad 1: +3V3 -> Net-(C24-Pad1)
- R32 pad 2: FSW2_SIG -> Net-(J8-Pin_2)
Routing:
- net PUMP1_GATE: track 12.0 -> 0.00 mm
- net VPMP_EN: track 8.36 -> 0.00 mm
- net VPLUG: track 6.19 -> 0.00 mm
- net VPMP: track 4.49 -> 0.00 mm
- net Net-(Q2-D): track 4.08 -> 0.00 mm
- net Net-(Q6-G): track 2.86 -> 0.00 mm
- net Net-(U5-VCP): track 2.14 -> 0.00 mm
- net +3V3: track 5.91 -> 4.03 mm
- net Net-(U5-5VOUT): track 1.85 -> 0.17 mm
- net Net-(U5-CPO): track 1.43 -> 0.00 mm
- net Net-(U5-CPI): track 1.41 -> 0.00 mm
- net Net-(U5-BRB): track 1.26 -> 0.00 mm
- net Net-(U5-BRA): track 1.24 -> 0.00 mm
- net Net-(Q4-G): track 1.17 -> 0.01 mm
- net S3_TXD: track 1.78 -> 0.69 mm
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
Commit message: LAYOUT work
Parts:
- removed C33: 0.1uF, Capacitor_SMD:C_0402_1005Metric
- removed Q6: DMN3032LE-13, DMN3032LE-13:SOT230P700X180-4N
- added C25: 10uF, Capacitor_SMD:C_0402_1005Metric, F.Cu at (104.8, 82.2)
- added C28: 0.1uF, Capacitor_SMD:C_0402_1005Metric, B.Cu at (129.6, 83.7)
- added C29: 0.1uF, Capacitor_SMD:C_0402_1005Metric, B.Cu at (129.6, 79.7)
- added Q1: AO3407A, Package_TO_SOT_SMD:SOT-23, F.Cu at (104.3, 84.8)
- added Q3: ZXMN3A01ZTA, ZXMN3A01ZTA:ZXMN3_DIO, F.Cu at (132.8, 72.5)
- added R36: 200, Resistor_SMD:R_0402_1005Metric, F.Cu at (103.3, 87.8)
- added R37: 13k, Resistor_SMD:R_0402_1005Metric, B.Cu at (132.0, 87.8)
- added R38: 20K, Resistor_SMD:R_0402_1005Metric, B.Cu at (130.0, 87.7)
- added R39: 1k, Resistor_SMD:R_0402_1005Metric, B.Cu at (129.6, 81.7)
- added R40: 1k, Resistor_SMD:R_0402_1005Metric, B.Cu at (129.6, 77.6)
- BZ1, C21, C24, C32, D13, Q5, R16, R19, R26, R27, R28, R32, R8, TP13, TP7: moved to B.Cu
- D6: footprint LED_SMD:LED_0805_2012Metric -> LED_SMD:LED_0603_1608Metric
- Q4: value DMN3032LE-13 -> ZXMN3A01ZTA; footprint DMN3032LE-13:SOT230P700X180-4N -> ZXMN3A01ZTA:ZXMN3_DIO
- R11: value 47k -> 20K; moved to B.Cu
- moved C21 139.8 mm to (183.9, 53.0), turned to 180 degrees
- moved Q5 125.5 mm to (183.6, 48.7), turned to 180 degrees
- moved TP2 115.3 mm to (163.0, 67.0)
- moved D8 109.8 mm to (174.7, 66.3), turned to 90 degrees
- moved R13 109.6 mm to (172.2, 64.8)
- moved R19 109.5 mm to (180.0, 43.0), turned to 180 degrees
- moved D7 105.6 mm to (169.7, 66.3), turned to 90 degrees
- moved R12 105.5 mm to (166.9, 64.7), turned to 180 degrees
- moved D10 105.4 mm to (165.0, 66.5), turned to 90 degrees
- moved R16 104.6 mm to (174.7, 41.2), turned to 180 degrees
- moved TP9 100.7 mm to (172.2, 66.8)
- moved R15 99.9 mm to (163.1, 65.4), turned to 180 degrees
- moved D13 98.7 mm to (175.1, 47.2), turned to 180 degrees
- moved TP5 96.2 mm to (167.2, 66.8)
- moved BZ1 93.9 mm to (172.7, 53.0), turned to 180 degrees
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Connections:
- C24 pad 1: Net-(C24-Pad1) -> FSW2_SIG
- C24 pad 2: FSW2_SIG -> GND
- C26 pad 2: +3V3 -> VSMS
- C32 pad 1: Net-(C32-Pad1) -> GND
- J6 pad 2: +3V3 -> VSMS
- J6 pad 3: SMS1_DATA -> Net-(J6-Pin_3)
- J6 pad 4: SMS2_DATA -> Net-(J6-Pin_4)
- J7 pad 3: I2C_DTA -> I2C_CLK
- J7 pad 4: I2C_CLK -> I2C_DTA
- Q4 pad 2: PUMP1_N -> PUMP2_N
- R22 pad 2: Net-(Q4-G) -> Net-(Q3-G)
- R23 pad 2: Net-(Q4-G) -> Net-(Q3-G)
- R24 pad 2: Net-(Q6-G) -> Net-(Q4-G)
- R25 pad 2: Net-(Q6-G) -> Net-(Q4-G)
- R27 pad 1: Net-(C32-Pad1) -> FSW1_SIG
- R32 pad 1: Net-(C24-Pad1) -> FSW2_SIG
- R33 pad 2: FSW1_SIG -> Net-(Q1-G)
- U4 pad 12: unconnected-(U4-IO8-Pad12) -> SMS1_DATA
- U4 pad 13: unconnected-(U4-IO19-Pad13) -> USB_N
- U4 pad 14: unconnected-(U4-IO20-Pad14) -> USB_P
- U4 pad 17: unconnected-(U4-IO9-Pad17) -> SMS2_DATA
- U4 pad 4: unconnected-(U4-IO4-Pad4) -> VCC_SENSE
- U4 pad 5: unconnected-(U4-IO5-Pad5) -> VPLUG_SENSE
- U4 pad 6: USB_N -> unconnected-(U4-IO6-Pad6)
- U4 pad 7: USB_P -> unconnected-(U4-IO7-Pad7)
Routing:
- net S3_BOOT: track 0.00 -> 7.92 mm
- net USB_P: track 18.7 -> 24.5 mm
- net USB_N: track 17.9 -> 23.5 mm
- net VCC_SENSE: track 0.00 -> 4.13 mm, vias 0 -> 1
- net VPLUG_SENSE: track 0.00 -> 4.03 mm, vias 0 -> 1
- net S3_EN: track 21.6 -> 24.1 mm
- net VSMS: track 0.00 -> 0.65 mm
Other:
- board text added: "homectrl"
- board text added: "jeevan sanchez || 2026"
- board text added: "model 2.0"

Commit message: power routing
Parts:
- BZ1, C28, C29, R11, R37, R38, R39, R40, R8: moved to F.Cu
- R2: footprint Resistor_SMD:R_0805_2012Metric -> Resistor_SMD:R_0603_1608Metric
- moved R25 33.2 mm to (137.8, 71.8), turned to 90 degrees
- moved R24 31.6 mm to (137.3, 70.1), turned to 0 degrees
- moved C31 7.53 mm to (148.1, 60.2), turned to -150 degrees
- moved R40 4.94 mm to (126.5, 81.4)
- moved R39 4.16 mm to (126.5, 84.5)
- moved Q3 4.03 mm to (134.1, 76.4)
- moved C22 4.03 mm to (141.2, 76.1)
- moved C18 4.03 mm to (142.5, 76.8)
- moved U8 3.99 mm to (147.1, 58.5), turned to 120 degrees
- moved C29 2.68 mm to (127.6, 81.4), turned to -90 degrees
- moved FB1 2.60 mm to (142.3, 42.6)
- moved C41 2.58 mm to (142.1, 45.2), turned to -90 degrees
- moved Q4 2.33 mm to (141.2, 71.6)
- moved C2 2.23 mm to (143.7, 45.6)
- moved R11 2.12 mm to (132.1, 85.2), turned to 180 degrees
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Connections:
- D1 pad 2: Net-(D1-A2) -> GND
- J1 pad 2: Net-(D1-A2) -> GND
- R2 pad 2: Net-(D1-A2) -> GND
Routing:
- net 5V_MUX: track 0.00 -> 25.6 mm
- net 5V_PLUG: track 0.00 -> 24.2 mm
- net GND: track 3.73 -> 26.0 mm, vias 1 -> 109
- net VPLUG: track 0.00 -> 14.8 mm
- net Net-(D4-K): track 0.00 -> 13.6 mm
- net +3V3: track 4.03 -> 17.4 mm
- net Net-(U1-COMP): track 0.00 -> 3.35 mm
- net 5V_USB: track 0.00 -> 3.12 mm
- net Net-(U1-BOOT): track 0.00 -> 2.16 mm
- net Net-(U1-ROSC): track 0.00 -> 1.80 mm
- net Net-(U1-SS): track 0.00 -> 1.80 mm
- net Net-(C8-Pad1): track 0.00 -> 1.06 mm
- added copper zone on F.Cu, net GND
- added copper zone on F.Cu, net Net-(D1-A1)
- added copper zone on F.Cu, net Net-(D3-K)
- added copper zone on F.Cu, net Net-(F1-Pad1)

Commit message: actuator routes
Parts:
- C31, U8: moved to B.Cu
- Q3: renamed from Q4; footprint ZXMN3A01ZTA:ZXMN3_DIO -> Package_TO_SOT_SMD:SOT-89-3
- Q4: renamed from Q3; footprint ZXMN3A01ZTA:ZXMN3_DIO -> Package_TO_SOT_SMD:SOT-89-3
- moved TP13 37.1 mm to (158.0, 44.3)
- moved TP7 37.1 mm to (160.5, 44.3)
- moved R25 9.20 mm to (146.9, 71.0), turned to 180 degrees
- moved R24 8.10 mm to (145.2, 71.5), turned to 90 degrees
- moved R23 4.67 mm to (126.6, 74.0)
- moved R22 4.67 mm to (126.1, 72.4)
- moved C29 2.99 mm to (130.1, 83.1)
- moved R40 2.99 mm to (129.0, 83.1)
- moved U8 2.09 mm to (146.3, 56.5)
- moved C31 2.06 mm to (147.3, 58.3)
- moved U3 1.51 mm to (133.2, 69.9)
- moved R6 1.48 mm to (129.0, 73.0)
- moved Q2 1.48 mm to (129.3, 69.9)
- moved R7 1.48 mm to (128.0, 73.0)
- moved Q4 1.07 mm to (133.3, 75.6)
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Connections:
- C24 pad 1: FSW2_SIG -> Net-(C24-Pad1)
- C32 pad 2: FSW1_SIG -> Net-(C32-Pad2)
- D1 pad 2: GND -> Net-(D1-A2)
- J1 pad 2: GND -> Net-(D1-A2)
- J4 pad 1: STEP_1A -> STEP_2A
- J4 pad 2: STEP_1B -> STEP_2B
- J4 pad 3: STEP_2A -> STEP_1A
- J4 pad 4: STEP_2B -> STEP_1B
- J8 pad 1: Net-(J8-Pin_1) -> FSW1_SIG
- J8 pad 2: Net-(J8-Pin_2) -> FSW2_SIG
- Q3 pad 1: Net-(Q4-G) -> Net-(Q3-G)
- Q3 pad 2: PUMP2_N -> PUMP1_N
- Q4 pad 1: Net-(Q3-G) -> Net-(Q4-G)
- Q4 pad 2: PUMP1_N -> PUMP2_N
- R2 pad 2: GND -> Net-(D1-A2)
- R26 pad 2: Net-(J8-Pin_1) -> FSW1_SIG
- R27 pad 1: FSW1_SIG -> Net-(C32-Pad2)
- R27 pad 2: Net-(J8-Pin_1) -> FSW1_SIG
- R28 pad 2: Net-(J8-Pin_2) -> FSW2_SIG
- R32 pad 1: FSW2_SIG -> Net-(C24-Pad1)
- R32 pad 2: Net-(J8-Pin_2) -> FSW2_SIG
Routing:
- net VPMP: track 0.00 -> 44.5 mm, vias 0 -> 3
- net STEP_2B: track 0.00 -> 33.5 mm, vias 0 -> 2
- net VPLUG: track 14.8 -> 44.2 mm, vias 0 -> 2
- net PUMP2_N: track 0.00 -> 25.1 mm
- net STEP_1A: track 0.00 -> 19.7 mm
- net PUMP1_N: track 0.00 -> 19.1 mm
- net STEP_1B: track 0.00 -> 18.8 mm
- net GND: track 26.0 -> 43.7 mm, vias 109 -> 142
- net MTR_STEP: track 0.00 -> 16.5 mm, vias 0 -> 2
- net MTR_DIR: track 0.00 -> 16.5 mm
- net STEP_2A: track 0.00 -> 16.2 mm
- net S3_RXD: track 0.00 -> 8.39 mm
- net Net-(D1-A2): track 0.00 -> 8.32 mm
- net S3_TXD: track 0.69 -> 8.32 mm
- net STEP_DIAG: track 0.00 -> 5.05 mm
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