File: hardware/homectrl-v2/homectrl-v2.kicad_pcb (KiCad board)
At the start: 4 copper layers, 64 x 70.5 mm, 133 parts, among them J1 Barrel_Jack, J2 PUMP1_CONN, J3 PUMP2_CONN, J4 STEP_CONN, J5 USB_C_CONN, J6 SMS1_CONN, J7 ALS_CONN, J8 FSW1_CONN, Q1 AO3407A, Q2 2N7002, Q3 AO3400A, Q4 AO3400A, Q5 AO3400A, SW1 S3_RESET_SW, SW2 S3_BOOT_SW, U1 TPS5405DR, U2 MCP1826S, U3 DMP4065S-7, U4 ESP32-S3-WROOM-1, U5 TMC2209, U7 TPD4E001DRLR, U8 TPD2E001DRLR, U9 SI2347DS-T1-GE3

Commit message: start silkscreen
Parts:
- added ?: , clipboard:fc8df92e-a3b3-4f73-a46e-2aabbf2af471, B.Cu at (112.2, 31.8)
- added G***: LOGO, LOGO, B.Cu at (145.9, 72.3)
- added G***: LOGO, LOGO, B.Cu at (122.2, 40.3)
- moved C20 0.29 mm to (127.2, 59.5)
- moved D14 0.29 mm to (124.6, 61.1)
Routing:
- net GND: track 149.9 -> 159.3 mm, vias 215 -> 209
- net Net-(J6-Pin_4): track 65.7 -> 67.0 mm
- net Net-(J6-Pin_3): track 66.4 -> 65.3 mm
- net STEP_2B: track 33.5 -> 34.4 mm
- net +3V3: track 211.2 -> 211.8 mm
Other:
- board text added: "+"
- board text added: "1"
- board text added: "2"
- board text added: "ESP32-S3 core integrated WiFi & BLE"
- board text added: "HI"
- board text added: "LO"
- board text added: "PCB: 4L FR4, 1.6mm, HASL"
- board text added: "PLG"
- board text added: "app"
- board text added: "boot"
- board text added: "bzz"
- board text added: "git"
- board text added: "jeevansanchez.com"
- board text added: "june 2026"
- board text added: "platform"
- board text added: "power 12V 2A"
- board text added: "reset"

Commit message: silkscreen
Parts:
- added ?: , clipboard:fc8df92e-a3b3-4f73-a46e-2aabbf2af471, B.Cu at (133.2, 98.4)
- added H1: MountingHole, MountingHole:MountingHole_2.2mm_M2, F.Cu at (100.2, 52.7)
- added H2: MountingHole, MountingHole:MountingHole_2.2mm_M2, F.Cu at (148.3, 84.0)
- C11, C16: footprint Capacitor_SMD:C_0402_1005Metric -> Capacitor_SMD:C_0603_1608Metric
- C25: value 10uF -> 0.1uF
- TP5: value TestPoint_Pad_D1.0mm -> VPLUG_TP_PAD
- moved C11 1.03 mm to (115.4, 51.3), turned to -90 degrees
- moved C16 0.54 mm to (127.6, 90.7)
- moved C10 0.32 mm to (115.5, 53.4)
- moved C14 0.18 mm to (126.4, 90.3)
- moved TP5 0.09 mm to (131.9, 45.2)
Routing:
- net GND: track 159.3 -> 161.2 mm, vias 209 -> 201
- net 5V_MUX: track 25.6 -> 27.0 mm
- net +3V3: track 211.8 -> 213.1 mm
- net Net-(J5-CC2): track 1.71 -> 2.84 mm
- net STEP_2A: track 14.6 -> 15.3 mm
Other:
- board text added: "ALS"
- board text added: "FSW"
- board text added: "PMP1"
- board text added: "PMP2"
- board text added: "SMS"
- board text added: "STP"
- board text added: "USBC"
- board text added: "modular automation"
- board text added: "smart irrigation blind control"

Commit message: prod
Parts:
- added TP7: VPLUG_TP_PAD, TestPoint:TestPoint_Pad_1.0x1.0mm, B.Cu at (141.9, 43.9)
- added TP9: GND_B_PAD, TestPoint:TestPoint_Pad_1.0x1.0mm, B.Cu at (129.7, 44.0)
- D7, R12: moved to B.Cu
- TP5: value VPLUG_TP_PAD -> VPLUG_TP_DRILL; footprint TestPoint:TestPoint_Pad_D1.0mm -> TestPoint:TestPoint_THTPad_D1.0mm_Drill0.5mm; moved to B.Cu
- moved TP5 8.19 mm to (140.0, 43.9), turned to 180 degrees
- moved R12 8.12 mm to (140.0, 42.6)
- moved D7 8.10 mm to (137.2, 42.6)
- moved R2 7.58 mm to (131.7, 45.4), turned to -90 degrees
- moved D3 3.15 mm to (129.6, 44.6), turned to -90 degrees
- moved C10 0.18 mm to (115.7, 53.4)
- moved J8 0.08 mm to (150.3, 55.6)
Connections:
- D1 pad 2: Net-(D1-A2) -> GND
- D3 pad 2: GND -> Net-(D3-A)
- J1 pad 2: Net-(D1-A2) -> GND
- R2 pad 2: Net-(D1-A2) -> Net-(D3-A)
- U9 pad 1: GND -> Net-(D3-A)
Routing:
- net Net-(D1-A2): track 8.32 -> 0.00 mm
- net Net-(D3-A): track 0.00 -> 5.67 mm
- net GND: track 161.2 -> 164.5 mm, vias 201 -> 253
- net +3V3: track 213.1 -> 211.3 mm
- net 5V_USB: track 67.8 -> 66.6 mm
- net Net-(Q2-D): track 12.5 -> 11.8 mm
- removed copper zone on F.Cu, net Net-(D1-A2)
Other:
- board text added: "S3"
- board text added: "barrel"
- board text added: "github"
- board text added: "type c"
- board text removed: "PCB: 4L FR4, 1.6mm, HASL"
- board text removed: "git"

Commit message: prods
Other:
- board text added: "5V"
- board text added: "5VP"
- board text added: "5VU"
- board text added: "BUCK"
- board text added: "LDO"
- board text added: "MUX"

Commit message: cleanup
Routing:
- net GND: track 164.5 -> 165.8 mm, vias 253 -> 254
Changed lines of the file:
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@@
+	)
+	(segment
+		(start 137.9511 66.7789)
+		(end 137.9511 67.0061)
+		(width 0.3)
+		(layer "F.Cu")
+		(net 3)
 	)
 	(segment
@@
 		(end 139.515 72.915)
 		(width 0.5)
+		(layer "F.Cu")
+		(net 3)
+	)
+	(segment
+		(start 138.75 65.98)
+		(end 137.9511 66.7789)
+		(width 0.3)
 		(layer "F.Cu")
 		(net 3)
@@
 		(net 3)
 	)
+	(via
+		(at 138.75 65.98)
+		(size 0.6)
+		(drill 0.3)
+		(layers "F.Cu" "B.Cu")
+		(net 3)
+	)
