File: hardware/homectrl-v2/_autosave-homectrl-v2.kicad_pcb (KiCad board)
At the start: 2 copper layers, 64 x 64 mm, 136 parts, among them J1 Barrel_Jack, J2 PUMP1_CONN, J3 PUMP2_CONN, J4 STEP_CONN, J5 USB_C_CONN, J6 SMS1_CONN, J7 ALS_CONN, J8 FSW1_CONN, Q1 AO3407A, Q2 2N7002, Q3 ZXMN3A01ZTA, Q4 ZXMN3A01ZTA, Q5 AO3400A, SW1 S3_RESET_SW, SW2 S3_BOOT_SW, U1 TPS5405DR, U2 MCP1826S, U3 DMP4065S-7, U4 ESP32-S3-WROOM-1, U5 TMC2209, U7 TPD4E001DRLR, U8 TPD2E001DRLR, U9 SI2347DS-T1-GE3

Commit message: misc work
Parts:
- removed R37: 13k, Resistor_SMD:R_0402_1005Metric
- removed R38: 20K, Resistor_SMD:R_0402_1005Metric
- added R22: 200, Resistor_SMD:R_0402_1005Metric, F.Cu at (140.8, 70.9)
- added R23: 10k, Resistor_SMD:R_0402_1005Metric, F.Cu at (141.3, 72.5)
- added REF**: SOT-23, Package_TO_SOT_SMD:SOT-23, F.Cu at (136.2, 78.2)
- added REF**: SOT-23, Package_TO_SOT_SMD:SOT-23, F.Cu at (143.8, 72.2)
- moved Q2 42.8 mm to (133.7, 72.2)
- moved R6 42.8 mm to (133.5, 75.2)
- moved R7 42.8 mm to (132.5, 75.2)
- moved U3 42.8 mm to (137.6, 72.1)
- moved R22 40.2 mm to (133.2, 76.9)
- moved R23 40.2 mm to (133.7, 78.5)
- moved C28 5.39 mm to (132.9, 83.5)
- moved R39 5.39 mm to (131.8, 83.5)
Connections:
- R22 pad 1: PUMP1_GATE -> PUMP1_EN
- R24 pad 1: PUMP2_GATE -> PUMP2_EN
- U4 pad 10: unconnected-(U4-IO17-Pad10) -> MTR_STEP
- U4 pad 11: unconnected-(U4-IO18-Pad11) -> MTR_DIR
- U4 pad 12: SMS1_DATA -> S3_RXD
- U4 pad 15: STEP_DIAG -> S3_TXD
- U4 pad 17: SMS2_DATA -> STEP_DIAG
- U4 pad 4: VCC_SENSE -> VPLUG_SENSE
- U4 pad 5: VPLUG_SENSE -> SMS1_DATA
- U4 pad 6: unconnected-(U4-IO6-Pad6) -> SMS2_DATA
- U4 pad 7: unconnected-(U4-IO7-Pad7) -> PUMP2_EN
- U4 pad 8: unconnected-(U4-IO15-Pad8) -> PUMP1_EN
- U4 pad 9: unconnected-(U4-IO16-Pad9) -> VPMP_EN
Routing:
- net MTR_STEP: track 25.7 -> 39.7 mm, vias 2 -> 4
- net MTR_DIR: track 26.6 -> 38.1 mm, vias 0 -> 2
- net S3_RXD: track 19.3 -> 28.7 mm, vias 0 -> 2
- net S3_TXD: track 20.0 -> 26.9 mm
- net VCC_SENSE: track 4.13 -> 0.00 mm, vias 1 -> 0
- net SMS1_DATA: track 0.00 -> 2.61 mm, vias 0 -> 1
- net S3_EN: track 24.1 -> 26.7 mm
- net STEP_DIAG: track 24.2 -> 26.8 mm
- net VPLUG_SENSE: track 4.03 -> 2.80 mm
